File: hardware/hardware.sch (KiCad schematic (older format))
At the start: 103 parts, among them J1 DB25_Female, J2 USB_B_Micro, J3 RJ45_Bel_SI-60062-F-68net, J4 Conn_01x02_Male, J5 Conn_01x02_Male, U1 MIC5319, U11 ENC28J60x-SO, U12 74LVC14, U2 74LVTH126, U3 74LVTH126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

Commit message: feat: update BOM
Parts:
- D1, D2: Digi-Key_PN 60-1456-1-ND -> 160-1456-1-ND
- J2: Digi-Key_PN 135698-ND -> A135698-ND
Changed lines of the file:
@@
 F 2 "kicad-footprints-perso:TE_2172034-1" H 1150 7200 50  0001 C CNN
 F 3 "~" H 1150 7200 50  0001 C CNN
-F 4 "135698-ND" H 1000 7250 50  0001 C CNN "Digi-Key_PN"
+F 4 "A135698-ND" H 1000 7250 50  0001 C CNN "Digi-Key_PN"
 F 5 "ok" H 1000 7250 50  0001 C CNN "checked"
 	1    1000 7250
@@
 F 2 "LED_SMD:LED_1206_3216Metric_Pad1.42x1.75mm_HandSolder" H 1650 9550 50  0001 C CNN
 F 3 "~" H 1650 9550 50  0001 C CNN
-F 4 "60-1456-1-ND" H 1650 9550 50  0001 C CNN "Digi-Key_PN"
+F 4 "160-1456-1-ND" H 1650 9550 50  0001 C CNN "Digi-Key_PN"
 F 5 "ok" H 1650 9550 50  0001 C CNN "checked"
 	1    1650 9550
@@
 F 2 "LED_SMD:LED_1206_3216Metric_Pad1.42x1.75mm_HandSolder" H 1650 10450 50  0001 C CNN
 F 3 "~" H 1650 10450 50  0001 C CNN
-F 4 "60-1456-1-ND" H 1650 10450 50  0001 C CNN "Digi-Key_PN"
+F 4 "160-1456-1-ND" H 1650 10450 50  0001 C CNN "Digi-Key_PN"
 F 5 "ok" H 1650 10450 50  0001 C CNN "checked"
 	1    1650 10450

Commit message: feat: update BOM
Parts:
- R17, R18, R19, R20: Digi-Key_PN RNCF0805DTE2K32CT-ND -> RNCF0805DTE49R9CT-ND
Changed lines of the file:
@@
 F 2 "Resistor_SMD:R_0805_2012Metric_Pad1.15x1.40mm_HandSolder" V 11280 7650 50  0001 C CNN
 F 3 "~" H 11350 7650 50  0001 C CNN
-F 4 "RNCF0805DTE2K32CT-ND" H 11350 7650 50  0001 C CNN "Digi-Key_PN"
+F 4 "RNCF0805DTE49R9CT-ND" H 11350 7650 50  0001 C CNN "Digi-Key_PN"
 F 5 "ok" H 11350 7650 50  0001 C CNN "checked"
 	1    11350 7650
@@
 F 2 "Resistor_SMD:R_0805_2012Metric_Pad1.15x1.40mm_HandSolder" V 10980 7650 50  0001 C CNN
 F 3 "~" H 11050 7650 50  0001 C CNN
-F 4 "RNCF0805DTE2K32CT-ND" H 11050 7650 50  0001 C CNN "Digi-Key_PN"
+F 4 "RNCF0805DTE49R9CT-ND" H 11050 7650 50  0001 C CNN "Digi-Key_PN"
 F 5 "ok" H 11050 7650 50  0001 C CNN "checked"
 	1    11050 7650
@@
 F 2 "Resistor_SMD:R_0805_2012Metric_Pad1.15x1.40mm_HandSolder" V 11280 8950 50  0001 C CNN
 F 3 "~" H 11350 8950 50  0001 C CNN
-F 4 "RNCF0805DTE2K32CT-ND" H 11350 8950 50  0001 C CNN "Digi-Key_PN"
+F 4 "RNCF0805DTE49R9CT-ND" H 11350 8950 50  0001 C CNN "Digi-Key_PN"
 F 5 "ok" H 11350 8950 50  0001 C CNN "checked"
 	1    11350 8950
@@
 F 2 "Resistor_SMD:R_0805_2012Metric_Pad1.15x1.40mm_HandSolder" V 10980 8950 50  0001 C CNN
 F 3 "~" H 11050 8950 50  0001 C CNN
-F 4 "RNCF0805DTE2K32CT-ND" H 11050 8950 50  0001 C CNN "Digi-Key_PN"
+F 4 "RNCF0805DTE49R9CT-ND" H 11050 8950 50  0001 C CNN "Digi-Key_PN"
 F 5 "ok" H 11050 8950 50  0001 C CNN "checked"
 	1    11050 8950
